File: KiCAD/LME49600_HPA/LME49600_HPA.kicad_pcb (KiCad board)
At the start: 2 copper layers, 81.3 x 88.9 mm, 55 parts, among them J1 PWR_IN, J2 IN_L, J3 OUT_L, J4 IN_R, J5 OUT_R, U1 NJM4580, U2 LME49600, U3 NJM4580, U4 LME49600

Commit message: Add: PCM2704 HPA ブロック図.xlsx
Parts:
- moved J2 10.8 mm to (144.8, 61.0), turned to 0 degrees
- moved J4 10.8 mm to (180.3, 61.0), turned to 0 degrees
- moved JP4 1.27 mm to (175.3, 101.6)
Routing:
- net GNDA: track 454.7 -> 1.25 mm
- net Net-(JP4-Pad1): track 5.27 -> 4.00 mm
- net -9V: track 203.2 -> 204.1 mm
Other:
- board text added: "LME49600 HPA V2.1"
- board text removed: "LME49600 HPA V2"
